File: ConsorcioMedico_Refrigeradora.kicad_sch (KiCad schematic)
At the start: 0 parts

Commit message: SCH: Se añadió el uC, pulsadores, display, fuente, relays (aunque falta escoger el correcto)
Parts:
- added C13: 10uF, 1-Capacitor:C_1206_3216Metric, symbol 1-Capacitor:C_1206
- added C44 (x2): 100nF 50V, 1-Capacitor:C_0805_2012Metric, symbol 1-Capacitor:C_0805
- added C45 (x4), C?: 1uF 50V, 1-Capacitor:C_0603_1608Metric, symbol 1-Capacitor:C_0603
- added C8: 1uF 10V, 1-Capacitor:C_0805_2012Metric, symbol 1-Capacitor:C_0805
- added C9: 4.7uF 5V, 1-Capacitor:C_0805_2012Metric, symbol 1-Capacitor:C_0805
- added C? (x4): 10nF 50V, 1-Capacitor:C_0603_1608Metric, symbol 1-Capacitor:C_0603
- added C?: 2.2uF 50V, 1-Capacitor:C_0603_1608Metric, symbol 1-Capacitor:C_0603
- added C? (x2): 15pF 10V, 1-Capacitor:C_0603_1608Metric, symbol 1-Capacitor:C_0603
- added C? (x2): 30pF 50V, 1-Capacitor:C_0603_1608Metric, symbol 1-Capacitor:C_0603
- added C? (x7): 100nF 50V, 1-Capacitor:C_0603_1608Metric, symbol 1-Capacitor:C_0603
- added D27 (x2), D6: RED, 1-Led:LED_0805, symbol 1-Led:LED_0805
- added D7, D8: 1N4148WS, Diode_SMD:D_SOD-323, symbol Diode:1N4148WS
- added J1: BatteryHolder, 1-Battery:BatteryHolder_DS1092_04_B6P, symbol Connector:Screw_Terminal_01x02
- added J3, J5: Screw_Terminal_01x01, 1-Pad:PAD_D2.60mm_Drill1.4mm, symbol Connector:Screw_Terminal_01x01
- added J37: SWD, Connector_PinHeader_2.54mm:PinHeader_1x06_P2.54mm_Vertical, symbol Connector:Screw_Terminal_01x06
- added J5: USART, 1-Pinhead:PinHeader_1x04_P2.54mm_Vertical, symbol Connector:Screw_Terminal_01x04
- added J5, J6: Screw_Terminal_01x03, 1-Terminal-Block:DG128_01x03_5.0P_10.5x15.5mm, symbol Connector:Screw_Terminal_01x03
- added J? (x2): Screw_Terminal_01x02, 1-Terminal-Block:DG504-5.08-02P_or_SMKDS 2,5-2-5.08, symbol 1-Terminal-Block:DG504-5.08-02P
- added K1: Q1, 1-Relay:Relay_DPDT_29mmX12.7mmX15.7mm, symbol 1-Relay:DPDT_29x12.5x15.7
- added K2: Q2, 1-Relay:Relay_DPDT_29mmX12.7mmX15.7mm, symbol 1-Relay:DPDT_29x12.5x15.7
- added LED1: LFD080AUE-103A-0, 1-Display:LFD080AUE-103A-0, symbol 1-Display:LFD080AUE-103A-0
- added Q1, Q2, Q3, Q4: MMBT3904, Package_TO_SOT_SMD:SOT-23, symbol Transistor_BJT:MMBT3904
- added Q1, Q2: BSS123, Package_TO_SOT_SMD:SOT-23, symbol Transistor_FET:BSS123
- added R10, R11, R12, R13, R14, R7, R8, R9: 120R, 1-Resistor:R_0603_1608Metric, symbol 1-Resistor:R_0603
- added R15, R16, R17, R18, R19, R20, R?: 10k, 1-Resistor:R_0603_1608Metric, symbol 1-Resistor:R_0603
- added R15, R17: 220R, 1-Resistor:R_0805_2012Metric, symbol 1-Resistor:R_0805
- added R16, R18: 10K, 1-Resistor:R_0805_2012Metric, symbol 1-Resistor:R_0805
- added R167 (x2): 3.9k, 1-Resistor:R_0805_2012Metric, symbol 1-Resistor:R_0805
- added R169 (x4): 1k, 1-Resistor:R_0805_2012Metric, symbol 1-Resistor:R_0805
- added R176 (x2): 2.7k, 1-Resistor:R_0805_2012Metric, symbol 1-Resistor:R_0805
- added R2, R209 (x2), R4, R5, R6: 1k, 1-Resistor:R_0603_1608Metric, symbol 1-Resistor:R_0603
- added R6: 680R, 1-Resistor:R_0603_1608Metric, symbol 1-Resistor:R_0603
- added S1: Buzz, 1-Switch:SW_PUSH-12mm-H, symbol 1-Switch:SW_PUSH_12mm_H
- added S2: Touch, 1-Switch:SW_PUSH-12mm-H, symbol 1-Switch:SW_PUSH_12mm_H
- added S3: Up, 1-Switch:SW_PUSH-12mm-H, symbol 1-Switch:SW_PUSH_12mm_H
- added S4: Down, 1-Switch:SW_PUSH-12mm-H, symbol 1-Switch:SW_PUSH_12mm_H
- added S5: Cooling, 1-Switch:SW_PUSH-12mm-H, symbol 1-Switch:SW_PUSH_12mm_H
- added S6: Light, 1-Switch:SW_PUSH-12mm-H, symbol 1-Switch:SW_PUSH_12mm_H
- added U1: STM32F411RETx, Package_QFP:LQFP-64_10x10mm_P0.5mm, symbol MCU_ST_STM32F4:STM32F411RETx
- added U13 (x2): INA350, 1-Package_TO_SOT_SMD:SOT-23-8, symbol 1-IC-Amplifier:INA350_SOT-23-8
- added U2: IRM-02, 1-Supply_Module-Eagle:IRM-02, symbol 1-Supply_Module-Eagle:IRM-02
- added U3: LDL1117, Package_TO_SOT_SMD:SOT-223-3_TabPin2, symbol Regulator_Linear:AMS1117
- added Y?: 8Mhz, 1-Crystal-and-Oscillator:Crystal_SMD_5032-2Pin_5.0x3.2mm, symbol Device:Crystal_Small
- added Y?: 32.768khz/12.5pF, 1-Crystal-and-Oscillator:Crystal_SMD_3215-2P_32.768khz, symbol Device:Crystal_Small
Connections:
- new net: J?.1 (Pin_1), R167.2, R169.1 (x2)
- new net: C45.1, R169.2, U13.3 (+) (x2)
- new net: D27.2 (A), R209.2 (x2)
- new net: J5.2 (Pin_2), K1.11
- new net: J5.3 (Pin_3), K1.12
- new net: J5.1 (Pin_1), K1.14
- new net: D7.2 (A), K1.2, Q1.3 (D)
- new net: Q2.1 (G), R17.2, R18.2
- new net: D8.2 (A), K2.2, Q2.3 (D)
- new net: LED1.5 (D), R10.2
- new net: LED1.8 (F), R12.2
- new net: C?.1, U1.30 (VCAP1)
- new net: C?.1, U1.4 (PC15), Y?.1
- new net: LED1.7 (E), R11.2
- new net: C?.1, U1.6 (PH1), Y?.2
- new net: J3.1 (Pin_1), U2.AC1
- new net: J5.1 (Pin_1), U2.AC2
- new net: C?.1, U1.3 (PC14), Y?.2
- new net: C?.1, U1.5 (PH0), Y?.1
- new net: R?.1, U1.60 (BOOT0)
- new net: C45.1, R169.2, U13.2 (-) (x2)
- new net: LED1.4 (B), R8.2
- new net: LED1.11 (A), R7.2
- new net: J?.2 (Pin_2), R169.1, R176.1 (x2)
- new net: Q2.1 (B), R4.2
- new net: LED1.3 (DIG2), Q2.3 (C)
- new net: D6.2 (A), R6.2
- new net: Q1.1 (G), R15.2, R16.2
- new net: LED1.9 (G), R13.2
- new net: Q1.1 (B), R2.2
- new net: LED1.1 (DIG1), Q1.3 (C)
- new net: LED1.10 (DIG3), Q3.3 (C)
- new net: LED1.12 (DIG4), Q4.3 (C)
- new net: LED1.2 (C), R9.2
- new net: LED1.6 (DP), R14.2
- new net: Q4.1 (B), R6.2
- new net: J6.2 (Pin_2), K2.21
- new net: J6.3 (Pin_3), K2.22
- new net: J6.1 (Pin_1), K2.24
- new net: Q3.1 (B), R5.2
- new net +3.3V: C44.1, C44.1, C9.1, C?.1, C?.1, C?.1, C?.1, C?.1, C?.1, C?.1, C?.1, C?.1, C?.1, J37.1 (Pin_1), J5.1 (Pin_1), R15.2, R16.2, R167.1, R167.1, R17.2, R18.2, R19.2, R20.2, U1.13 (VDDA), U1.19 (VDD), U1.32 (VDD), U1.48 (VDD), U1.64 (VDD), U13.7 (V+), U13.7 (V+), U3.2 (VO)
- new net +5V: C13.1, C8.1, D7.1 (K), D8.1 (K), K1.1, K2.1, U2.+V (+), U3.3 (VI)
- new net +BATT: C?.1, J1.1 (Pin_1), U1.1 (VBAT)
- new net A: R7.1, U1.14 (PA0)
- new net B: R8.1, U1.15 (PA1)
- new net Button_Buzzer: R17.1, S1.1, U1.55 (PB3)
- new net Button_Cooling: R19.1, S5.1, U1.59 (PB7)
- new net Button_Down: R18.1, S4.1, U1.58 (PB6)
- new net Button_Light: R20.1, S6.1, U1.61 (PB8)
- new net Button_Touch: R15.1, S2.1, U1.56 (PB4)
- new net Button_Up: R16.1, S3.1, U1.57 (PB5)
- new net C: R9.1, U1.16 (PA2)
- new net D: R10.1, U1.17 (PA3)
- new net DIG1: R2.1, U1.41 (PA8)
- new net DIG2: R4.1, U1.42 (PA9)
- new net DIG3: R5.1, U1.43 (PA10)
- new net DIG4: R6.1, U1.44 (PA11)
- new net DP: R14.1, U1.23 (PA7)
- new net E: R11.1, U1.20 (PA4)
- new net F: R12.1, U1.21 (PA5)
- new net G: R13.1, U1.22 (PA6)
- new net GND: C13.2, C44.2, C44.2, C45.2, C45.2, C45.2, C45.2, C8.2, C9.2, C?.2, C?.2, C?.2, C?.2, C?.2, C?.2, C?.2, C?.2, C?.2, C?.2, C?.2, C?.2, C?.2, C?.2, C?.2, C?.2, C?.2, D27.1 (K), D27.1 (K), D6.1 (K), J1.2 (Pin_2), J37.3 (Pin_3), J5.4 (Pin_4), Q1.2 (E), Q1.2 (S), Q2.2 (E), Q2.2 (S), Q3.2 (E), Q4.2 (E), R16.1, R176.2, R176.2, R18.1, R?.2, S1.3, S1.4, S2.3, S2.4, S3.3, S3.4, S4.3, S4.4, S5.3, S5.4, S6.3, S6.4, U1.12 (VSSA), U1.18 (VSS), U1.31 (VSS), U1.47 (VSS), U1.63 (VSS), U13.4 (V-), U13.4 (V-), U13.5 (REF), U13.5 (REF), U2.-V (-), U3.1 (ADJ)
- new net MCU_RX6: J5.2 (Pin_2)
- new net MCU_TX6: J5.3 (Pin_3)
- new net RELAY_Q1: R15.1
- new net RELAY_Q2: R17.1
- new net RESET: C?.1, J37.5 (Pin_5), U1.7 (NRST)
- new net RTD1: R209.1, U13.6
- new net RTD2: R209.1, U13.6
- new net STATUS_LED: R6.1
- new net SWCLK: J37.2 (Pin_2)
- new net SWDIO: J37.4 (Pin_4)
- new net SWO: J37.6 (Pin_6)
- no-connect marks 0 -> 10
Other:
- note added: "0.05V"
- note added: "1V"
- note added: "ANALOG"
- note added: "BUTTONS"
- note added: "Battery"
- note added: "COMM"
- note added: "DISPLAY"
- note added: "Fuente de voltaje"
- note added: "Internal Pull-Up"
- note added: "JTAG/SWD"
- note added: "MCU"
- note added: "NOTES"
- note added: "POWER SUPPLY"
- note added: "RELAY Q1"
- note added: "RELAY Q2"
- note added: "RTD: PT100 I = 500uA"
- note added: "STM32F411RET6: C94355 Crystal 8Mhz: C115962"
- note added: "Status Led"
- note added: "TestPoint:TestPoint_Loop_D2.60mm_Drill1.4mm_Beaded"
- note added: "USART"
- note added: "VDD y VSS"
- note added: "VDDA"

Commit message: Commit de guardado
Parts:
- added D7: 1N4148WS, Diode_SMD:D_SOD-323, symbol Diode:1N4148WS
- added D7, D8, D9: LED_RECT, 1-Led:LED_3.9x1.9mm, symbol 1-Led:LED_0805
- added J5: Screw_Terminal_01x03, 1-Terminal-Block:DG128_01x03_5.0P_10.5x15.5mm, symbol Connector:Screw_Terminal_01x03
- added K1: Q1, 1-Relay:Relay_DPDT_29mmX12.7mmX15.7mm, symbol 1-Relay:DPDT_29x12.5x15.7
- added Q1: BSS123, Package_TO_SOT_SMD:SOT-23, symbol Transistor_FET:BSS123
- added R15: 220R, 1-Resistor:R_0805_2012Metric, symbol 1-Resistor:R_0805
- added R16: 10K, 1-Resistor:R_0805_2012Metric, symbol 1-Resistor:R_0805
- added R6 (x3): 330, 1-Resistor:R_0603_1608Metric, symbol 1-Resistor:R_0603
- R6: value 680R -> 1000
Connections:
- net +5V: now also D7.1 (K), K1.1
- net GND: now also D7.1 (K), D8.1 (K), D9.1 (K), Q1.2 (S), R16.1
- net RELAY_Q1: now also R15.1
- net STATUS_LED: now also U1.33 (PB12), R6.1, R6.1, R6.1
- new net: D8.2 (A), R6.2
- new net: D9.2 (A), R6.2
- new net: D7.2 (A), K1.2, Q1.3 (D)
- new net: Q1.1 (G), R15.2, R16.2
- new net: J5.2 (Pin_2), K1.11
- new net: J5.3 (Pin_3), K1.12
- new net: J5.1 (Pin_1), K1.14
- new net: D7.2 (A), R6.2
- no-connect marks 10 -> 13
Other:
- note added: "LEDS"
- note added: "RELAY Q3"
- note removed: "Status Led"
- moved on the sheet: C44, C45, D27, D6, J37, J5, J?, LED1, Q1, Q2, Q3, Q4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

Commit message: SCH: Aún queda resolver la entrada digital para el switch y la fuente de voltaje. PCB: Se están acomodando los componentes
Parts:
- removed D6: RED, 1-Led:LED_0805, symbol 1-Led:LED_0805
- removed D7, D8: LED_RECT, 1-Led:LED_3.9x1.9mm, symbol 1-Led:LED_0805
- removed J5 (x2), J6: Screw_Terminal_01x03, 1-Terminal-Block:DG128_01x03_5.0P_10.5x15.5mm, symbol Connector:Screw_Terminal_01x03
- removed K1 (x2): Q1, 1-Relay:Relay_DPDT_29mmX12.7mmX15.7mm, symbol 1-Relay:DPDT_29x12.5x15.7
- removed K2: Q2, 1-Relay:Relay_DPDT_29mmX12.7mmX15.7mm, symbol 1-Relay:DPDT_29x12.5x15.7
- added D1, D7, D8: L-144IDT, 1-Led:LED_3.9x1.9mm, symbol 1-Led:LED_Rect
- added D8: 1N4148WS, Diode_SMD:D_SOD-323, symbol Diode:1N4148WS
- added J10, J11, J12, J13, J14, J15, J8, J9: Screw_Terminal_01x01, 1-Pad:PAD_D2.60mm_Drill1.4mm, symbol Connector:Screw_Terminal_01x01
- added K1, K3, K4: HF46F-G/012-HS1T, 1-Relay:Relay_HONGFA_SPST-NO_20.5x7x15.3mm, symbol 1-Relay:Relay_HONGFA_SPST-NO_20.5x7x15.3mm
- added K2: T9AS1D12-12, 1-Relay:Relay_TE-Connectivity_SPST-NO_32.5x27.4x27.9mm, symbol 1-Relay:Relay_TE_SPST-NO_32.5x27.4x27.9mm
- added Q2: BSS123, Package_TO_SOT_SMD:SOT-23, symbol Transistor_FET:BSS123
- added R17: 220R, 1-Resistor:R_0805_2012Metric, symbol 1-Resistor:R_0805
- added R18: 10K, 1-Resistor:R_0805_2012Metric, symbol 1-Resistor:R_0805
- D9: value LED_RECT -> LED_0805; footprint 1-Led:LED_3.9x1.9mm -> 1-Led:LED_0805
Connections:
- net RELAY_Q2 is gone; now on net Relay_Light: R17.1
- net +5V: now also D8.1 (K), K1.2, K2.2, K3.2, K4.2
- net DIG1: now also U1.11 (PC3); no longer U1.41 (PA8)
- net DIG2: now also U1.10 (PC2); no longer U1.42 (PA9)
- net DIG3: now also U1.9 (PC1); no longer U1.43 (PA10)
- net DIG4: now also U1.8 (PC0); no longer U1.44 (PA11)
- net GND: now also D1.K, D7.K, D8.K, Q2.2 (S), R18.1
- net at R6.2: now also D7.A
- net at D7.2 (A), Q1.3 (D): now also K1.1
- net at D8.2 (A), Q2.3 (D): now also K4.1
- net at D9.2 (A): now also R6.2; no longer R6.2
- net at D7.2 (A), Q1.3 (D): now also K2.1
- net Relay_Fan: now reaches U1.24 (PC4)
- net Relay_Fan: now also R15.1
- net Relay_Light: now reaches U1.25 (PC5)
- net Relay_Compressor: now reaches U1.37 (PC6)
- net Relay_Compressor: now also R15.1
- net Relay_Calefac: now reaches U1.38 (PC7)
- net Relay_Calefac: now also R17.1
- net LED_Status: now reaches U1.45 (PA12)
- net LED_Status: now also R6.1
- net LED_Defrost: now reaches U1.46 (PA13)
- net LED_Defrost: now also R6.1
- net LED_Door: now reaches U1.49 (PA14)
- net LED_Door: now also R6.1
- net LED_TempAlarm: now reaches U1.50 (PA15)
- net LED_TempAlarm: now also R6.1
- net at R6.2: now also D1.A
- removed net RELAY_Q1: R15.1, R15.1
- removed net STATUS_LED: R6.1, R6.1, R6.1, R6.1, U1.33 (PB12)
- new net: D8.2 (A), K3.1, Q2.3 (D)
- new net: J15.1 (Pin_1), K3.3
- new net: J14.1 (Pin_1), K3.4
- new net: J10.1 (Pin_1), K4.4
- new net: Q2.1 (G), R17.2, R18.2
- new net: J13.1 (Pin_1), K2.3
- new net: J12.1 (Pin_1), K2.4
- new net: D8.A, R6.2
- new net: J9.1 (Pin_1), K1.3
- new net: J8.1 (Pin_1), K1.4
- new net: J11.1 (Pin_1), K4.3
- no-connect marks 13 -> 4
Other:
- note added: "Potencia: 12V 720R = 16mA 12V 144R = 83mA 3x16 + 83 = 131mA -> Potencia regulador: 12V*131mA = 1.57W"
- note added: "Relay Compressor + Condensador"
- note added: "Relay Luz"
- note added: "Relay Resistencia"
- note added: "Relay Ventilador del Evaporador"
- note added: "Relay originales: HF46F 12-HS 12V Coil 5A 250VAC: https://www.tme.com/pe/es/details/hf46f_012-hs1/reles-electromagn-miniaturizados/hongfa-relay/hf46f-12-hs1/ HF32F-G 012-HST 12V Coil 10A 250VAC:http://www.hongfaamerica.com/hq/PDF/HF32F-G_en.pdf HF2150-1A-12DE: https://es.aliexpress.com/item/1000009105435.html Relay Remplazo: HF46F-G/012-HS1T 12V Coil 10A 250VAC https://www.tme.com/pe/es/details/h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"
- note removed: "RELAY Q1"
- note removed: "RELAY Q2"
- note removed: "RELAY Q3"
- note removed: "TestPoint:TestPoint_Loop_D2.60mm_Drill1.4mm_Beaded"
- moved on the sheet: C?, D7, D8, J1, J37, J5, Q1, Q2, R15, R16, R17, R18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
