File: ConsorcioMedico_Refrigeradora.kicad_pcb (KiCad board)
At the start: 2 copper layers, 260 x 70 mm, 156 parts, among them J1 BatteryHolder, J10 AC, J11 Digital, J12 Light, J13 Light, J14 Compress, J15 Resistor, J16 Analog, J18 Resistor, J19 AC, J2 USART, J3 USART, J4 SWD, J5 Evap_fan, J6 Screw_Terminal_01x01, J7 Screw_Terminal_01x01, J8 Evap_fan, J9 Compress, K1 HF46F-G/012-HS1T, K2 AZ2150-1A-12DEF, K3 HF46F-G/012-HS1T, K4 HF46F-G/012-HS1T, Q1 MMBT3904, Q11 BSS806, Q2 MMBT3904, Q3 MMBT3904, Q4 MMBT3904, Q5 BSS806, Q6 BSS806, Q7 BSS806, Q8 BSS806, Q9 BSS806, U1 STM32F411RETx, U2 AP63205WU, U3 LDL1117, U4 INA350, U5 INA350, U6 LTV-357T, U7 LTV-357T, U9 HLK-PMx, Y1 8Mhz, Y2 32.768khz/12.5pF

Commit message: SCH: pin EN se corrige para activar la alimentación de 5V, se cambia el empaquetado de varias resistencias 0603 a 0805. PCB: Se alarga el plano de GND, se acomodan los componentes 0805, se completa de colocar la serigrafía, se ensancha la pista de AC. JLCPCB: Se actualiza
Parts:
- R1, R10, R11, R12, R13, R14, R15, R16, R17, R18, R19, R2, R20, R24, R29, R35, R36, R38, R4, R5, R6, R7, R8, R9: footprint 1-Resistor:R_0603_1608Metric -> 1-Resistor:R_0805_2012Metric
- moved R24 6.78 mm to (117.6, 123.9), turned to -90 degrees
- moved R29 4.01 mm to (115.1, 123.9), turned to -90 degrees
- moved R20 1.71 mm to (263.5, 108.6)
- moved R17 0.54 mm to (161.4, 108.6)
- moved R16 0.42 mm to (130.8, 108.3)
- moved R7 0.30 mm to (60.3, 97.0)
- moved R36 0.22 mm to (63.3, 99.7)
- moved R15 0.21 mm to (209.7, 108.6)
- moved D1 0.20 mm to (48.3, 124.9)
- moved R12 0.20 mm to (48.3, 97.0)
- moved R38 0.11 mm to (69.7, 99.6)
- moved R1 0.10 mm to (50.4, 124.8)
- moved R19 0.10 mm to (234.0, 108.4)
- moved R14 0.10 mm to (38.8, 99.6)
- moved R18 0.10 mm to (184.4, 108.4)
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Connections:
- U2 pad 2: GND -> +12V
Routing:
- net GND: track 500.9 -> 465.7 mm, vias 67 -> 104
- net I2C3_SCL: track 42.2 -> 56.6 mm
- net I2C3_SDA: track 42.1 -> 47.0 mm
- net Button_Light: track 215.7 -> 217.4 mm
- net Relay_On: track 59.4 -> 60.7 mm
- net Button_Up: track 135.2 -> 136.4 mm
- net Button_Down: track 158.3 -> 159.4 mm
- net RTD1: track 48.3 -> 47.3 mm
- net +12V: track 409.1 -> 410.1 mm
- net Button_Buzzer: track 69.8 -> 69.1 mm
- net Button_Cooling: track 186.9 -> 187.6 mm
- net RTD2: track 37.1 -> 36.4 mm
- net DIG4: track 28.7 -> 28.0 mm
- net +3.3V: track 495.7 -> 495.9 mm, vias 51 -> 57
Other:
- board text added: "AC1"
- board text added: "AC2"
- board text added: "AN0"
- board text added: "AN1"
- board text added: "BUZZER"
- board text added: "COMPRESSOR"
- board text added: "COOLING"
- board text added: "DOWN"
- board text added: "FAN"
- board text added: "I0"
- board text added: "I1"
- board text added: "LIGHT"
- board text added: "RESISTOR"
- board text added: "TOUCH"
- board text added: "UP"
