File: Dig_Inputs.kicad_sch (KiCad schematic)
At the start: 31 parts, among them J11 Digital, U3 LTV-357T

Commit message: SCH: pin EN se corrige para activar la alimentación de 5V, se cambia el empaquetado de varias resistencias 0603 a 0805. PCB: Se alarga el plano de GND, se acomodan los componentes 0805, se completa de colocar la serigrafía, se ensancha la pista de AC. JLCPCB: Se actualiza
Parts:
- R15, R16, R17, R18, R19, R20: footprint 1-Resistor:R_0603_1608Metric -> 1-Resistor:R_0805_2012Metric
Changed lines of the file:
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@@
       (effects (font (size 1.27 1.27)) (justify right))
     )
-    (property "Footprint" "1-Resistor:R_0603_1608Metric" (at 175.768 48.26 90)
+    (property "Footprint" "1-Resistor:R_0805_2012Metric" (at 175.768 48.26 90)
       (effects (font (size 1.27 1.27)) hide)
     )
@@
       (effects (font (size 1.27 1.27)) (justify right))
     )
-    (property "Footprint" "1-Resistor:R_0603_1608Metric" (at 255.778 87.63 90)
+    (property "Footprint" "1-Resistor:R_0805_2012Metric" (at 255.778 87.63 90)
       (effects (font (size 1.27 1.27)) hide)
     )
@@
       (effects (font (size 1.27 1.27)) (justify right))
     )
-    (property "Footprint" "1-Resistor:R_0603_1608Metric" (at 249.428 48.26 90)
+    (property "Footprint" "1-Resistor:R_0805_2012Metric" (at 249.428 48.26 90)
       (effects (font (size 1.27 1.27)) hide)
     )
@@
       (effects (font (size 1.27 1.27)) (justify right))
     )
-    (property "Footprint" "1-Resistor:R_0603_1608Metric" (at 215.138 87.63 90)
+    (property "Footprint" "1-Resistor:R_0805_2012Metric" (at 215.138 87.63 90)
       (effects (font (size 1.27 1.27)) hide)
     )
@@
       (effects (font (size 1.27 1.27)) (justify right))
     )
-    (property "Footprint" "1-Resistor:R_0603_1608Metric" (at 175.768 87.63 90)
+    (property "Footprint" "1-Resistor:R_0805_2012Metric" (at 175.768 87.63 90)
       (effects (font (size 1.27 1.27)) hide)
     )
@@
       (effects (font (size 1.27 1.27)) (justify right))
     )
-    (property "Footprint" "1-Resistor:R_0603_1608Metric" (at 212.598 48.26 90)
-      (effects (font (size 1.27 1.27)) hide)
-    )
+    (property "Footprint" "1-Resistor:R_0805_2012Metric" (at 212.598 48.26 90)
+      (effects (font (size 1.27 1.27)) hide)
+    )

Commit message: SCH
Connections:
- net Button_Cooling is gone; now on net Button_Light: R19.1, S5.1
- net Button_Light: no longer R20.1, S6.1
- net Button_Buzzer renamed Button_Power
- net Button_Touch renamed Button_Set
- new net Button_Sound: R20.1, S6.1
Changed lines of the file:
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@@
     (effects (font (size 5 5) (thickness 1) bold) (justify left bottom))
-  )
-  (global_label "Button_Cooling" (shape input) (at 209.55 93.98 180) (fields_autoplaced)
-    (effects (font (size 1 1)) (justify right))
-    (property "Intersheetrefs" "${INTERSHEET_REFS}" (at 196.0238 93.98 0)
-      (effects (font (size 1.27 1.27)) (justify right) hide)
-    )
   )
   (global_label "DIG_IN_0" (shape input) (at 93.98 45.72 0) (fields_autoplaced)
@@
     )
   )
+  (global_label "Button_Set" (shape input) (at 243.84 54.61 180) (fields_autoplaced)
+    (effects (font (size 1 1)) (justify right))
+    (property "Intersheetrefs" "${INTERSHEET_REFS}" (at 233.5521 54.61 0)
+      (effects (font (size 1.27 1.27)) (justify right) hide)
+    )
+  )
   (global_label "I0" (shape output) (at 118.11 50.8 270) (fields_autoplaced)
     (effects (font (size 1.27 1.27)) (justify right))
     (property "Intersheetrefs" "${INTERSHEET_REFS}" (at 118.11 55.5201 90)
+      (effects (font (size 1.27 1.27)) (justify right) hide)
+    )
+  )
+  (global_label "Button_Power" (shape input) (at 207.01 54.61 180) (fields_autoplaced)
+    (effects (font (size 1 1)) (justify right))
+    (property "Intersheetrefs" "${INTERSHEET_REFS}" (at 194.6745 54.61 0)
       (effects (font (size 1.27 1.27)) (justify right) hide)
     )
@@
     )
   )
+  (global_label "Button_Sound" (shape input) (at 250.19 93.98 180) (fields_autoplaced)
+    (effects (font (size 1 1)) (justify right))
+    (property "Intersheetrefs" "${INTERSHEET_REFS}" (at 237.7114 93.98 0)
+      (effects (font (size 1.27 1.27)) (justify right) hide)
+    )
+  )
   (global_label "DIG_IN_1" (shape input) (at 95.25 97.79 0) (fields_autoplaced)
     (effects (font (size 1 1)) (justify left))
@@
     )
   )
-  (global_label "Button_Touch" (shape input) (at 243.84 54.61 180) (fields_autoplaced)
+  (global_label "Button_Light" (shape input) (at 209.55 93.98 180) (fields_autoplaced)
     (effects (font (size 1 1)) (justify right))
-    (property "Intersheetrefs" "${INTERSHEET_REFS}" (at 231.5996 54.61 0)
+    (property "Intersheetrefs" "${INTERSHEET_REFS}" (at 197.9763 93.98 0)
       (effects (font (size 1.27 1.27)) (justify right) hide)
     )
@@
     (effects (font (size 1 1)) (justify right))
     (property "Intersheetrefs" "${INTERSHEET_REFS}" (at 158.4158 54.61 0)
-      (effects (font (size 1.27 1.27)) (justify right) hide)
-    )
-  )
-  (global_label "Button_Buzzer" (shape input) (at 207.01 54.61 180) (fields_autoplaced)
-    (effects (font (size 1 1)) (justify right))
-    (property "Intersheetrefs" "${INTERSHEET_REFS}" (at 194.1031 54.61 0)
       (effects (font (size 1.27 1.27)) (justify right) hide)
     )
@@
       (effects (font (size 1.27 1.27)) (justify right) hide)
     )
-  )
-  (global_label "Button_Light" (shape input) (at 250.19 93.98 180) (fields_autoplaced)
-    (effects (font (size 1 1)) (justify right))
-    (property "Intersheetrefs" "${INTERSHEET_REFS}" (at 238.6163 93.98 0)
-      (effects (font (size 1.27 1.27)) (justify right) hide)
-    )

Commit message: Luego de modificaciones de Dandy
Parts:
- added C35: 1uF 50V, 1-Capacitor:C_0805_2012Metric, symbol 1-Capacitor:C_0805
- added JP3: SolderJumper_3_Open, 1-Jumper:SolderJumper-3_P1.3mm_Open_RoundedPad1.0x1.5mm, symbol Jumper:SolderJumper_3_Open
- added R64: 1k, 1-Resistor:R_0805_2012Metric, symbol 1-Resistor:R_0805
- R15: value 10k -> 22k
Connections:
- net +12V: now also JP3.1 (A)
- net Button_Down: now also C35.1, R64.1; no longer R15.1, S1.1
- net GND: now also C35.2, JP3.3 (B); no longer J11.2 (Pin_2), J11.4 (Pin_4)
- new net: R15.1, R64.2, S1.1
- new net: J11.2 (Pin_2), J11.4 (Pin_4), JP3.2 (C)
Other:
- moved on the sheet: C30, C33, D10, D7, J11, JP1, JP2, R10, R13, R15, R16, R17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
